File: pi-jtag-adapter.kicad_pcb (KiCad board)
At the start: 2 copper layers, 16 x 53 mm, 6 parts, among them J1 Raspberry_Pi, J2 SWD, J3 UART, J4 UART

Commit message: Fix the layout
Parts:
- JP1, JP2: moved to B.Cu
- moved JP2 4.81 mm to (96.2, 63.5), turned to 90 degrees
- moved JP1 1.41 mm to (93.5, 63.5), turned to 90 degrees
Routing:
- net /TMS: track 16.3 -> 23.7 mm
- net GND: track 0.00 -> 4.32 mm
- net /RPI_RX: track 65.7 -> 61.7 mm, vias 1 -> 0
- net /DBG_RX: track 10.1 -> 13.3 mm
- net /TDO: track 18.1 -> 21.0 mm, vias 2 -> 1
- net /RPI_TX: track 56.1 -> 58.5 mm, vias 0 -> 1
- net /nRST: track 6.67 -> 8.59 mm, vias 0 -> 1
- net /DBG_TX: track 15.3 -> 13.9 mm
- net +3.3V: track 65.9 -> 64.6 mm
- net /TDI: track 28.3 -> 27.4 mm, vias 2 -> 1
Other:
- board text added: "Raspberry Pi Debug Adapter v1.1 Ilya Strukov 2024"
- board text removed: "Raspberry Pi Debug Adapter v1.0 Ilya Strukov 2024"

Commit message: Fix schematic and PCB layout
Connections:
- J1 pad 12: /TDO -> unconnected-(J1-GPIO18/PWM0-Pad12)
- J1 pad 18: unconnected-(J1-GPIO24-Pad18) -> /TDO
- J2 pad 10: /TMS -> /nRST
- J2 pad 2: /nRST -> /TMS
- J2 pad 4: /TDI -> /TCK
- J2 pad 8: /TCK -> /TDI
Routing:
- net /TMS: track 23.7 -> 10.3 mm, vias 2 -> 1
- net /nRST: track 8.59 -> 19.6 mm
- net /TDO: track 21.0 -> 10.6 mm, vias 1 -> 0
- net /TCK: track 8.84 -> 11.5 mm, vias 0 -> 1
- net /TDI: track 27.4 -> 24.8 mm
Other:
- board text added: "39"
