File: pi-jtag-adapter.kicad_sch (KiCad schematic)
At the start: 6 parts, among them J1 Raspberry_Pi, J2 SWD, J3 UART, J4 UART

Commit message: Fix schematic and PCB layout
Connections:
- net TCK: now also J2.4 (Pin_4); no longer J2.8 (Pin_8)
- net TDI: now also J2.8 (Pin_8); no longer J2.4 (Pin_4)
- net TDO: now also J1.18 (GPIO24); no longer J1.12 (GPIO18/PWM0)
- net TMS: now also J2.2 (Pin_2); no longer J2.10 (Pin_10)
- net nRST: now also J2.10 (Pin_10); no longer J2.2 (Pin_2)
- no-connect marks 23 -> 22
Changed lines of the file:
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@@
   (no_connect (at 133.35 67.31))
   (no_connect (at 173.99 92.71))
-  (no_connect (at 133.35 90.17))
   (no_connect (at 173.99 77.47))
   (no_connect (at 173.99 72.39))
   (no_connect (at 133.35 77.47))
+  (wire (pts (xy 115.57 90.17) (xy 76.2 90.17))
+    (stroke (width 0) (type default))
+  )
   (wire (pts (xy 49.53 59.69) (xy 49.53 95.25))
     (stroke (width 0) (type default))
@@
     (stroke (width 0) (type default))
   )
-  (wire (pts (xy 76.2 95.25) (xy 97.79 95.25))
-    (stroke (width 0) (type default))
-  )
   (wire (pts (xy 102.87 48.26) (xy 130.81 48.26))
-    (stroke (width 0) (type default))
-  )
-  (wire (pts (xy 101.6 87.63) (xy 101.6 85.09))
     (stroke (width 0) (type default))
   )
@@
     (stroke (width 0) (type default))
   )
-  (wire (pts (xy 101.6 85.09) (xy 133.35 85.09))
+  (wire (pts (xy 120.65 90.17) (xy 120.65 91.44))
+    (stroke (width 0) (type default))
+  )
+  (wire (pts (xy 127 97.79) (xy 127 87.63))
+    (stroke (width 0) (type default))
+  )
+  (wire (pts (xy 113.03 91.44) (xy 113.03 92.71))
+    (stroke (width 0) (type default))
+  )
+  (wire (pts (xy 123.19 85.09) (xy 133.35 85.09))
+    (stroke (width 0) (type default))
+  )
+  (wire (pts (xy 76.2 97.79) (xy 123.19 97.79))
     (stroke (width 0) (type default))
   )
@@
     (stroke (width 0) (type default))
   )
+  (wire (pts (xy 123.19 85.09) (xy 123.19 97.79))
+    (stroke (width 0) (type default))
+  )
   (wire (pts (xy 158.75 113.03) (xy 161.29 113.03))
     (stroke (width 0) (type default))
@@
     (stroke (width 0) (type default))
   )
-  (wire (pts (xy 76.2 87.63) (xy 101.6 87.63))
-    (stroke (width 0) (type default))
-  )
   (wire (pts (xy 63.5 97.79) (xy 46.99 97.79))
-    (stroke (width 0) (type default))
-  )
-  (wire (pts (xy 88.9 69.85) (xy 133.35 69.85))
     (stroke (width 0) (type default))
   )
@@
     (stroke (width 0) (type default))
   )
-  (wire (pts (xy 76.2 90.17) (xy 102.87 90.17))
+  (wire (pts (xy 127 87.63) (xy 76.2 87.63))
     (stroke (width 0) (type default))
   )
-  (wire (pts (xy 88.9 92.71) (xy 88.9 69.85))
-    (stroke (width 0) (type default))
-  )
-  (wire (pts (xy 76.2 97.79) (xy 133.35 97.79))
-    (stroke (width 0) (type default))
-  )
-  (wire (pts (xy 102.87 90.17) (xy 102.87 95.25))
+  (wire (pts (xy 120.65 91.44) (xy 113.03 91.44))
     (stroke (width 0) (type default))
   )
   (wire (pts (xy 46.99 48.26) (xy 92.71 48.26))
+    (stroke (width 0) (type default))
+  )
+  (wire (pts (xy 115.57 92.71) (xy 115.57 90.17))
     (stroke (width 0) (type default))
   )
@@
     (stroke (width 0) (type default))
   )
+  (wire (pts (xy 133.35 97.79) (xy 127 97.79))
+    (stroke (width 0) (type default))
+  )
   (wire (pts (xy 156.21 113.03) (xy 158.75 113.03))
     (stroke (width 0) (type default))
   )
-  (wire (pts (xy 102.87 95.25) (xy 133.35 95.25))
+  (wire (pts (xy 76.2 95.25) (xy 133.35 95.25))
     (stroke (width 0) (type default))
   )
@@
     (stroke (width 0) (type default))
   )
-  (wire (pts (xy 97.79 95.25) (xy 97.79 92.71))
+  (wire (pts (xy 133.35 90.17) (xy 120.65 90.17))
     (stroke (width 0) (type default))
   )
-  (wire (pts (xy 76.2 92.71) (xy 88.9 92.71))
+  (wire (pts (xy 76.2 92.71) (xy 113.03 92.71))
     (stroke (width 0) (type default))
   )
-  (wire (pts (xy 97.79 92.71) (xy 133.35 92.71))
+  (wire (pts (xy 115.57 92.71) (xy 133.35 92.71))
     (stroke (width 0) (type default))
   )
@@
     (effects (font (size 1.27 1.27)) (justify left bottom))
   )
-  (label "nRST" (at 76.2 87.63 0) (fields_autoplaced)
+  (label "nRST" (at 76.2 97.79 0) (fields_autoplaced)
     (effects (font (size 1.27 1.27)) (justify left bottom))
   )
@@
     (effects (font (size 1.27 1.27)) (justify left bottom))
   )
-  (label "TDI" (at 76.2 90.17 0) (fields_autoplaced)
+  (label "TDI" (at 76.2 95.25 0) (fields_autoplaced)
     (effects (font (size 1.27 1.27)) (justify left bottom))
   )
@@
     (effects (font (size 1.27 1.27)) (justify left bottom))
   )
-  (label "TCK" (at 76.2 95.25 0) (fields_autoplaced)
+  (label "TCK" (at 76.2 90.17 0) (fields_autoplaced)
     (effects (font (size 1.27 1.27)) (justify left bottom))
   )
@@
     (effects (font (size 1.27 1.27)) (justify left bottom))
   )
-  (label "TMS" (at 76.2 97.79 0) (fields_autoplaced)
+  (label "TMS" (at 76.2 87.63 0) (fields_autoplaced)
     (effects (font (size 1.27 1.27)) (justify left bottom))
   )
